File: V2_WIP/gps.kicad_pcb (KiCad board)
At the start: 6 copper layers, 82.5 x 82.5 mm, 124 parts, among them J202 USB4145-03-0230-C, J301 USB_B_Micro, J601 BATT, Q1 IRLML5203, Q2 S8050, Q3 S8050, SW2 FSM14JLH, SW602 MSN22AFW01, SW701 RotaryEncoder, U1 ESP32-WROOM-32E, U102 W25Q128JFV, U11 SN74LV1T34DBVRG4, U14 CH340K, U2 TPS613222ADBVR, U201 RT9080, U301 USBLC6-2SC6, U4 HT16k33, U401 NEO-M9N, U402 KW4-804CGB, U5 7seg_1x1_rgb, U6 7seg_1x1_rgb, U601 IP5306, U602 STC3100IST, U7 7seg_1x1_rgb, U9 TCA39306DDFR

Commit message: minor changes
Parts:
- removed SW_RST201: FSM14JLH, Button_Switch_THT:SW_PUSH_6mm
- added C201: 22u, Capacitor_SMD:C_0603_1608Metric_Pad1.08x0.95mm_HandSolder, F.Cu at (143.3, 77.2)
- added C610: 470u, Capacitor_SMD:C_Elec_6.3x7.7, F.Cu at (147.7, 66.5)
- added R202: Manual rst, Resistor_SMD:R_0603_1608Metric_Pad0.98x0.95mm_HandSolder, F.Cu at (143.3, 79.7)
- added R_E605: 33mR, Resistor_SMD:R_0603_1608Metric_Pad0.98x0.95mm_HandSolder, F.Cu at (143.3, 72.6)
- C606: value 22u -> 10u; footprint Capacitor_SMD:C_0603_1608Metric_Pad1.08x0.95mm_HandSolder -> Capacitor_Tantalum_SMD:CP_EIA-3528-15_AVX-H_Pad1.50x2.35mm_HandSolder
- moved SW2 38.6 mm to (111.5, 115.4)
Connections:
- C603 pad 1: Net-(D601-K) -> /VBATT
- C606 pad 1: GND -> +5V
- C606 pad 2: +5V -> GND
- L601 pad 2: Net-(D601-K) -> /VBATT
- R_E603 pad 2: Net-(D601-K) -> /VBATT
- TP3 pad 1: /RGB -> /RGB_DATA
- U1 pad 16: /ESP/IO13 -> /RGB_DATA
- U11 pad 2: /RGB -> /RGB_DATA
- U601 pad 6: Net-(D601-K) -> /VBATT
Routing:
- net Net-(D601-K): track 7.11 -> 0.00 mm
- net /VBATT: track 1.81 -> 8.92 mm
- net Net-(R2-Pad2): track 6.50 -> 0.00 mm
- net /ESP/RST: track 15.9 -> 9.36 mm
- net GND: vias 130 -> 129
- net +5V: vias 10 -> 11
