File: V2_WIP/gps.kicad_pcb (KiCad board)
At the start: 6 copper layers, 82.5 x 82.5 mm, 127 parts, among them J202 USB4145-03-0230-C, J301 USB_B_Micro, J601 BATT, Q1 IRLML5203, Q2 S8050, Q3 S8050, SW2 FSM14JLH, SW602 MSN22AFW01, SW701 RotaryEncoder, U1 ESP32-WROOM-32E, U102 W25Q128JFV, U11 SN74LV1T34DBVRG4, U14 CH340K, U2 TPS613222ADBVR, U201 RT9080, U301 USBLC6-2SC6, U4 HT16k33, U401 NEO-M9N, U402 KW4-804CGB, U5 7seg_1x1_rgb, U6 7seg_1x1_rgb, U601 IP5306, U602 STC3100IST, U7 7seg_1x1_rgb, U9 TCA39306DDFR

Commit message: finallizes schematic; pcb progress
Parts:
- removed C1: 100n, Capacitor_SMD:C_0603_1608Metric_Pad1.08x0.95mm_HandSolder
- removed C102: 470u, Capacitor_SMD:C_0603_1608Metric_Pad1.08x0.95mm_HandSolder
- removed C4, C5, C6: 10uF, Capacitor_SMD:C_0603_1608Metric_Pad1.08x0.95mm_HandSolder
- removed D2: B120-E3, Diode_SMD:D_SMA
- removed L1: 2.2 uH, Inductor_SMD:L_1008_2520Metric_Pad1.43x2.20mm_HandSolder
- removed R1: 0R, Resistor_SMD:R_0805_2012Metric_Pad1.20x1.40mm_HandSolder
- removed TP5: +5V, TestPoint:TestPoint_Pad_D1.5mm
- removed U2: TPS613222ADBVR, Package_TO_SOT_SMD:SOT-23-5
- added C103: 100nF, Capacitor_SMD:C_0805_2012Metric_Pad1.18x1.45mm_HandSolder, B.Cu at (131.1, 67.2)
- added C104: 100nF, Capacitor_SMD:C_0805_2012Metric_Pad1.18x1.45mm_HandSolder, B.Cu at (128.0, 70.8)
- added C202: C_Polarized, Capacitor_SMD:C_Elec_6.3x7.7, B.Cu at (111.5, 71.4)
- added C404: 100nF, Capacitor_SMD:C_0805_2012Metric_Pad1.18x1.45mm_HandSolder, B.Cu at (104.2, 56.3)
- added C405: 100nF, Capacitor_SMD:C_0805_2012Metric_Pad1.18x1.45mm_HandSolder, B.Cu at (83.9, 56.5)
- added C406: 100nF, Capacitor_SMD:C_0805_2012Metric_Pad1.18x1.45mm_HandSolder, B.Cu at (69.2, 56.1)
- added C702: 1n, Capacitor_SMD:C_0603_1608Metric_Pad1.08x0.95mm_HandSolder, B.Cu at (66.9, 110.0)
- added C703: 1n, Capacitor_SMD:C_0603_1608Metric_Pad1.08x0.95mm_HandSolder, B.Cu at (66.9, 119.0)
- added D301: M2, Diode_SMD:D_SMA, B.Cu at (64.7, 103.8)
- added R203: 10k, Resistor_SMD:R_0603_1608Metric_Pad0.98x0.95mm_HandSolder, B.Cu at (128.1, 76.7)
- added R_E705: 47, Resistor_SMD:R_0603_1608Metric_Pad0.98x0.95mm_HandSolder, B.Cu at (66.9, 117.2)
- added R_E706: 47, Resistor_SMD:R_0603_1608Metric_Pad0.98x0.95mm_HandSolder, B.Cu at (66.9, 111.8)
- added TP102: IMU_INT, TestPoint:TestPoint_Pad_D1.5mm, B.Cu at (128.0, 62.8)
- added TP103: +5V, TestPoint:TestPoint_Pad_D1.5mm, B.Cu at (125.8, 56.2)
- added TP202: VCC, TestPoint:TestPoint_Pad_D1.5mm, B.Cu at (107.6, 75.1)
- added U103: ICM-45686, Package_LGA:LGA-14_3x2.5mm_P0.5mm_LayoutBorder3x4y, B.Cu at (128.0, 67.1)
- C201, R202, R_E605: moved to B.Cu
- C610: value 470u -> C_Polarized; moved to B.Cu
- D3, D4: value D -> M2; footprint Diode_SMD:D_0603_1608Metric_Pad1.05x0.95mm_HandSolder -> Diode_SMD:D_SMA
- D6, D7: value D -> 1N4148W-G3-08; footprint Diode_SMD:D_0603_1608Metric_Pad1.05x0.95mm_HandSolder -> Diode_SMD:D_SOD-123
- R102: value R_Photo -> NSL-A95011
- R103: value 6k -> 56k; moved to B.Cu
- SW2: footprint Button_Switch_THT:SW_PUSH_6mm -> Button_Switch_SMD:SW_SPST_PTS647_Sx38
- TP12: value IO22 -> IO12
- TP3: value RGB_3V3 -> RGB_DATA
- U1: value ESP32-WROOM-32E -> ESP32-WROOM-32UE
- U201: value RT9080 -> RT9080-33GJ5
- moved R10 57.4 mm to (72.5, 51.1), turned to 90 degrees
- moved C610 56.0 mm to (92.0, 61.0), turned to 90 degrees
- moved D201 53.6 mm to (75.5, 52.5), turned to 90 degrees
- moved SW2 42.1 mm to (128.1, 76.7)
- moved R102 38.0 mm to (111.7, 111.9)
- moved R103 38.0 mm to (113.3, 111.9)
- moved R202 35.9 mm to (122.4, 108.9), turned to 180 degrees
- moved TP201 35.7 mm to (107.7, 93.0)
- moved C201 29.4 mm to (115.6, 87.3)
- moved R_E605 28.1 mm to (117.6, 61.0), turned to 90 degrees
- moved TP602 17.0 mm to (116.3, 64.4)
- moved U602 17.0 mm to (113.9, 59.3)
- moved C608 17.0 mm to (113.4, 54.4)
- moved C609 17.0 mm to (117.6, 57.5)
- moved R_E604 17.0 mm to (113.1, 64.4)
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Connections:
- net /CS_N renamed /SEL_FL
- C610 pad 1: GND -> +5V
- C610 pad 2: +5V -> GND
- J301 pad 1: Net-(J301-VBUS) -> Net-(D301-A)
- R102 pad 1: +3V3 -> /LIGHT_SENS
- R102 pad 2: /LIGHT_SENS -> GND
- R103 pad 1: GND -> /LIGHT_SENS
- R103 pad 2: /LIGHT_SENS -> +3V3
- R2 pad 1: /ESP/IO27 -> /ESP/IO15
- SW701 pad A: /CLK -> Net-(R_E705-Pad2)
- SW701 pad B: /DT -> Net-(R_E706-Pad2)
- U1 pad 10: /CLK -> /SW
- U1 pad 11: /SW -> /CLK
- U1 pad 12: /ESP/IO27 -> /DT
- U1 pad 23: /DT -> /ESP/IO15
- U1 pad 29: /ESP/IO5 -> unconnected-(U1-IO5-Pad29)
- U1 pad 3: /ESP/EN -> /ESP/RST
- U1 pad 4: /ESP/SENSOR_VP -> unconnected-(U1-SENSOR_VP-Pad4)
- U1 pad 5: /ESP/SENSOR_VN -> unconnected-(U1-SENSOR_VN-Pad5)
- U1 pad 6: /ESP/IO34 -> unconnected-(U1-IO34-Pad6)
- U1 pad 8: unconnected-(U1-IO32-Pad8) -> /SEL_IMU
- U301 pad 5: Net-(J301-VBUS) -> Net-(D301-A)
- U4 pad 11: /Display/f -> unconnected-(U4-ROW14/K12-Pad11)
- U4 pad 12: /Display/a -> unconnected-(U4-ROW13/K11-Pad12)
- U4 pad 13: /Display/b -> unconnected-(U4-ROW12/K10-Pad13)
- U4 pad 15: /Display/e -> unconnected-(U4-ROW10/K8-Pad15)
- U4 pad 17: /Display/c -> unconnected-(U4-ROW8/K6-Pad17)
- U4 pad 18: unconnected-(U4-ROW7/K5-Pad18) -> /Display/DP
- U4 pad 19: /Display/d -> /Display/g
- U4 pad 2: /Display/CC3 -> /Display/CC11
- U4 pad 20: unconnected-(U4-ROW5/K3-Pad20) -> /Display/f
- U4 pad 21: unconnected-(U4-ROW4/K2-Pad21) -> /Display/e
- U4 pad 22: unconnected-(U4-ROW3/K1-Pad22) -> /Display/d
- U4 pad 23: unconnected-(U4-ROW2/A0-Pad23) -> /Display/c
- U4 pad 24: /Display/DP -> /Display/b
- U4 pad 25: /Display/g -> /Display/a
- U4 pad 3: /Display/CC44 -> /Display/CC22
- U4 pad 5: /Display/CC22 -> /Display/CC44
- U4 pad 6: /Display/CC2 -> /Display/CC1
- U4 pad 7: /Display/CC11 -> /Display/CC2
- U4 pad 8: /Display/CCL123 -> /Display/CC3
- U4 pad 9: /Display/CC1 -> /Display/CCL123
Routing:
- net /VUSB: track 91.9 -> 206.0 mm, vias 12 -> 21
- net /VBATT: track 8.92 -> 91.4 mm, vias 2 -> 4
- net /RGB_DATA: track 0.00 -> 77.9 mm, vias 0 -> 2
- net /SW: track 1.99 -> 73.8 mm, vias 1 -> 2
- net /Pulse: track 0.00 -> 70.1 mm, vias 1 -> 2
- net /ESP/D+: track 6.16 -> 75.9 mm
- net /ESP/D-: track 3.18 -> 69.1 mm
- net /ESP/IO2: track 0.00 -> 63.9 mm, vias 1 -> 2
- net /DT: track 6.25 -> 68.2 mm, vias 1 -> 2
- net /CLK: track 6.25 -> 68.2 mm, vias 1 -> 2
- net /SCL_3V3: track 6.22 -> 65.9 mm
- net /SDA_3V3: track 5.74 -> 60.3 mm
- net /GNSS_RxD: track 22.7 -> 71.2 mm
- net /SEL_IMU: track 0.00 -> 47.1 mm, vias 0 -> 2
- net Net-(R2-Pad2): track 0.00 -> 46.5 mm, vias 0 -> 2
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- added copper zone on B.Cu, net +5V
- removed copper zone on B.Cu, net Net-(D2-A)

Commit message: updated most datashets
Parts:
- removed TP603: +5V, TestPoint:TestPoint_Pad_D1.5mm
- C202, C610: moved to F.Cu
- moved C610 36.1 mm to (59.7, 77.1)
- moved C202 17.7 mm to (128.6, 67.0)
- moved TP103 16.5 mm to (109.3, 55.6)
- moved TP2 3.57 mm to (109.3, 62.0)
- moved TP402 3.48 mm to (80.3, 83.4)
- moved TP401 2.65 mm to (80.3, 80.6)
- moved TP102 2.63 mm to (130.6, 63.4)
- moved TP1 2.53 mm to (109.3, 58.9)
- moved D201 1.07 mm to (76.5, 52.0)
- moved R10 1.07 mm to (73.5, 50.6)
- moved TP202 0.20 mm to (107.4, 75.1)
Routing:
- net +5V: track 76.6 -> 94.9 mm, vias 12 -> 13
- net Net-(BT301-+): track 50.5 -> 62.6 mm
- net /GNSS_RxD: track 71.2 -> 60.8 mm
- net /DT: track 68.2 -> 59.4 mm
- net /SDA_3V3: track 60.3 -> 66.4 mm
- net /Display/c: track 37.2 -> 32.3 mm
- net /SCL_3V3: track 65.9 -> 68.8 mm
- net /Display/DP: track 38.0 -> 35.4 mm
- net +3V3: track 29.2 -> 27.1 mm, vias 20 -> 28
- net Net-(J301-D-): track 4.67 -> 6.70 mm
- net /CLK: track 68.2 -> 66.3 mm
- net /VUSB: track 206.0 -> 204.1 mm, vias 21 -> 20
- net /RGB_DATA: track 77.9 -> 79.7 mm, vias 2 -> 3
- net /GNSS_TxD: track 57.9 -> 59.5 mm
- net /SW: track 73.8 -> 72.5 mm
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- added copper zone on B.Cu, net +3V3

Commit message: up to date i dont remember what changed
Parts:
- added C203: 1uF, Capacitor_SMD:C_0603_1608Metric_Pad1.08x0.95mm_HandSolder, B.Cu at (130.4, 110.5)
- added C204: 10uF, Capacitor_SMD:C_0603_1608Metric_Pad1.08x0.95mm_HandSolder, B.Cu at (129.6, 108.9)
- C10, C101, C103, C104, C404, C405, C406, C7, C9: footprint Capacitor_SMD:C_0805_2012Metric_Pad1.18x1.45mm_HandSolder -> Capacitor_SMD:C_0603_1608Metric_Pad1.08x0.95mm_HandSolder
- C11, C3, C601, C602, C603, C604: value 10u -> 10uF
- C14, C15, C2, C608, C609, C701: value 100n -> 100nF
- C201, C605: value 22u -> 22uF
- C202, C610: value C_Polarized -> 470uF
- C401: value 10uF -> *10uF
- C403: value 10n -> 10nF
- C606: value 10u -> *10uF
- C702, C703: value 1n -> 1nF
- DS1: value LTC-4724JF -> *LTC-4724JF
- J301: value USB_B_Micro -> *USB_B_Micro
- L601: value 1uH -> *1uH
- R16: value 2k2 -> 2k
- R_E703: value 1k -> 2k
- SW2: value FSM14JLH -> PTS647SN70SMTR2N LFS
- SW701: value RotaryEncoder -> *RotaryEncoder
- U102: value W25Q128JFV -> *W25Q128JFV
- U11: value SN74LV1T34DBVRG4 -> *SN74LV1T34DBVRG4
- U14: value CH340K -> *CH340K
- U4: value HT16k33 -> *HT16k33
- U401: value NEO-M9N -> *NEO-M9N
- U402: value KW4-804CGB -> *KW4-804CGB
- U5, U6, U7: value 7seg_1x1_rgb -> *7seg_1x1_rgb
- U601: value IP5306 -> *IP5306
- U9: value TCA39306DDFR -> *TCA39306DDFR
Routing:
- net +3V3: track 27.1 -> 30.9 mm, vias 28 -> 29
- net /ESP/D-: track 69.9 -> 72.5 mm
- net /ESP/D+: track 76.6 -> 75.5 mm
- net /VBATT: track 91.6 -> 92.2 mm
- net GND: vias 203 -> 261
- added copper zone on In1.Cu, net GND
