File: V2_WIP/Display.kicad_sch (KiCad schematic)
At the start: 13 parts, among them U11 SN74LV1T34DBVRG4, U4 HT16k33, U402 KW4-804CGB, U5 7seg_1x1_rgb, U6 7seg_1x1_rgb, U7 7seg_1x1_rgb

Commit message: updated most datashets
Parts:
- C404, C405, C406, C7, C9: footprint Capacitor_SMD:C_0805_2012Metric_Pad1.18x1.45mm_HandSolder -> Capacitor_SMD:C_0603_1608Metric_Pad1.08x0.95mm_HandSolder
- DS1: value LTC-4724JF -> *LTC-4724JF
- U11: value SN74LV1T34DBVRG4 -> *SN74LV1T34DBVRG4
- U4: value HT16k33 -> *HT16k33
- U402: value KW4-804CGB -> *KW4-804CGB
- U5, U6, U7: value 7seg_1x1_rgb -> *7seg_1x1_rgb
Changed lines of the file:
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@@
 			)
 		)
-		(property "Value" "LTC-4724JF"
+		(property "Value" "*LTC-4724JF"
 			(at 100.33 130.81 0)
 			(effects
@@
 			)
 		)
+		(property "Purchase-URL" ""
+			(at 62.23 135.89 0)
+			(effects
+				(font
+					(size 1.27 1.27)
+				)
+				(hide yes)
+			)
+		)
 		(pin "15"
 		)
@@
 			)
 		)
-		(property "Value" "SN74LV1T34DBVRG4"
+		(property "Value" "*SN74LV1T34DBVRG4"
 			(at 213.36 137.16 0)
 			(effects
@@
 			)
 		)
+		(property "Purchase-URL" ""
+			(at 203.2 144.78 0)
+			(effects
+				(font
+					(size 1.27 1.27)
+				)
+				(hide yes)
+			)
+		)
 		(pin "4"
 		)
@@
 			)
 		)
+		(property "Purchase-URL" ""
+			(at 215.9 144.78 0)
+			(effects
+				(font
+					(size 1.27 1.27)
+				)
+				(hide yes)
+			)
+		)
 		(pin "1"
 		)
@@
 			)
 		)
-		(property "Footprint" "Capacitor_SMD:C_0805_2012Metric_Pad1.18x1.45mm_HandSolder"
+		(property "Footprint" "Capacitor_SMD:C_0603_1608Metric_Pad1.08x0.95mm_HandSolder"
 			(at 244.1448 113.03 0)
 			(effects
@@
 			)
 		)
-		(property "Datasheet" "~"
+		(property "Datasheet" "https://cz.mouser.com/ProductDetail/KYOCERA-AVX/0603ZG104ZAT2A?qs=XWDBCzcA0Tke70DI9cEVbA%3D%3D"
 			(at 245.11 116.84 0)
 			(effects
@@
 			)
 		)
+		(property "Purchase-URL" ""
+			(at 245.11 116.84 0)
+			(effects
+				(font
+					(size 1.27 1.27)
+				)
+				(hide yes)
+			)
+		)
 		(pin "1"
 		)
@@
 			)
 		)
-		(property "Value" "HT16k33"
+		(property "Value" "*HT16k33"
 			(at 100.33 49.53 0)
 			(effects
@@
 		)
 		(property "Description" ""
+			(at 100.33 76.2 0)
+			(effects
+				(font
+					(size 1.27 1.27)
+				)
+				(hide yes)
+			)
+		)
+		(property "Purchase-URL" ""
 			(at 100.33 76.2 0)
 			(effects
@@
 			)
 		)
-		(property "Value" "7seg_1x1_rgb"
+		(property "Value" "*7seg_1x1_rgb"
 			(at 235.204 137.16 0)
 			(effects
@@
 			)
 		)
+		(property "Purchase-URL" ""
+			(at 228.6 139.7 0)
+			(effects
+				(font
+					(size 1.27 1.27)
+				)
+				(hide yes)
+			)
+		)
 		(pin "1"
 		)
@@
 			)
 		)
-		(property "Footprint" "Capacitor_SMD:C_0805_2012Metric_Pad1.18x1.45mm_HandSolder"
+		(property "Footprint" "Capacitor_SMD:C_0603_1608Metric_Pad1.08x0.95mm_HandSolder"
 			(at 152.0952 67.31 0)
 			(effects
@@
 			)
 		)
-		(property "Datasheet" "~"
+		(property "Datasheet" "https://cz.mouser.com/ProductDetail/KYOCERA-AVX/0603ZG104ZAT2A?qs=XWDBCzcA0Tke70DI9cEVbA%3D%3D"
 			(at 151.13 63.5 0)
 			(effects
@@
 			)
 		)
+		(property "Purchase-URL" ""
+			(at 151.13 63.5 0)
+			(effects
+				(font
+					(size 1.27 1.27)
+				)
+				(hide yes)
+			)
+		)
 		(pin "1"
 		)
@@
 			)
 		)
-		(property "Value" "7seg_1x1_rgb"
+		(property "Value" "*7seg_1x1_rgb"
 			(at 251.968 137.16 0)
 			(effects
@@
 			)
 		)
+		(property "Purchase-URL" ""
+			(at 245.11 139.7 0)
+			(effects
+				(font
+					(size 1.27 1.27)
+				)
+				(hide yes)
+			)
+		)
 		(pin "1"
 		)
@@
 			)
 		)
-		(property "Footprint" "Capacitor_SMD:C_0805_2012Metric_Pad1.18x1.45mm_HandSolder"
+		(property "Footprint" "Capacitor_SMD:C_0603_1608Metric_Pad1.08x0.95mm_HandSolder"
 			(at 202.2348 113.03 0)
 			(effects
@@
 			)
 		)
-		(property "Datasheet" "~"
+		(property "Datasheet" "https://cz.mouser.com/ProductDetail/KYOCERA-AVX/0603ZG104ZAT2A?qs=XWDBCzcA0Tke70DI9cEVbA%3D%3D"
 			(at 203.2 116.84 0)
 			(effects
@@
 			)
 		)
+		(property "Purchase-URL" ""
+			(at 203.2 116.84 0)
+			(effects
+				(font
+					(size 1.27 1.27)
+				)
+				(hide yes)
+			)
+		)
 		(pin "1"
 		)
@@
 			)
 		)
-		(property "Footprint" "Capacitor_SMD:C_0805_2012Metric_Pad1.18x1.45mm_HandSolder"
+		(property "Footprint" "Capacitor_SMD:C_0603_1608Metric_Pad1.08x0.95mm_HandSolder"
 			(at 261.9248 113.03 0)
 			(effects
@@
 			)
 		)
-		(property "Datasheet" "~"
+		(property "Datasheet" "https://cz.mouser.com/ProductDetail/KYOCERA-AVX/0603ZG104ZAT2A?qs=XWDBCzcA0Tke70DI9cEVbA%3D%3D"
 			(at 262.89 116.84 0)
 			(effects
@@
 			)
 		)
+		(property "Purchase-URL" ""
+			(at 262.89 116.84 0)
+			(effects
+				(font
+					(size 1.27 1.27)
+				)
+				(hide yes)
+			)
+		)
 		(pin "1"
 		)
@@
 			)
 		)
-		(property "Value" "7seg_1x1_rgb"
+		(property "Value" "*7seg_1x1_rgb"
 			(at 270.002 136.906 0)
 			(effects
@@
 			)
 		)
+		(property "Purchase-URL" ""
+			(at 262.89 139.7 0)
+			(effects
+				(font
+					(size 1.27 1.27)
+				)
+				(hide yes)
+			)
+		)
 		(pin "1"
 		)
@@
 			)
 		)
-		(property "Footprint" "Capacitor_SMD:C_0805_2012Metric_Pad1.18x1.45mm_HandSolder"
+		(property "Footprint" "Capacitor_SMD:C_0603_1608Metric_Pad1.08x0.95mm_HandSolder"
 			(at 227.6348 113.03 0)
 			(effects
@@
 			)
 		)
-		(property "Datasheet" "~"
+		(property "Datasheet" "https://cz.mouser.com/ProductDetail/KYOCERA-AVX/0603ZG104ZAT2A?qs=XWDBCzcA0Tke70DI9cEVbA%3D%3D"
 			(at 228.6 116.84 0)
 			(effects
@@
 			)
 		)
+		(property "Purchase-URL" ""
+			(at 228.6 116.84 0)
+			(effects
+				(font
+					(size 1.27 1.27)
+				)
+				(hide yes)
+			)
+		)
 		(pin "1"
 		)
@@
 			)
 		)
-		(property "Value" "KW4-804CGB"
+		(property "Value" "*KW4-804CGB"
 			(at 100.33 96.52 0)
 			(effects
@@
 			(at 100.33 111.76 0)
 			(effects
+				(font
+					(size 1.27 1.27)
+				)
+				(hide yes)
+			)
+		)
+		(property "Purchase-URL" ""
+			(at 100.33 111.76 0)
+			(effects
