File: V2_WIP/Display.kicad_sch (KiCad schematic)
At the start: 13 parts, among them U11 *SN74LV1T34DBVRG4, U4 *HT16k33, U402 *KW4-804CGB, U5 *7seg_1x1_rgb, U6 *7seg_1x1_rgb, U7 *7seg_1x1_rgb

Commit message: updated list of changes in README.md
Parts:
- added D8: 1N4148W-G3-08, Diode_SMD:D_SOD-123, symbol Device:D
- added R_E103, R_E104, R_E105, R_E106, R_E107, R_E108, R_E109, R_E110: 0R, Resistor_SMD:R_0603_1608Metric_Pad0.98x0.95mm_HandSolder, symbol Device:R
- added R_E111, R_E112, R_E113: 39k, Resistor_SMD:R_0603_1608Metric_Pad0.98x0.95mm_HandSolder, symbol Device:R
- TP403: footprint TestPoint:TestPoint_Pad_D1.5mm -> TestPoint:TestPoint_Pad_D1.0mm
- U4: footprint w_smd_dil:soic-28 -> Package_SO:SOIC-28W_7.5x17.9mm_P1.27mm
Connections:
- net CC1: now also R_E104.1; no longer DS1.1 (COMMON_CATHODE_DIGIT_1)
- net CC11: now also D8.2 (A), R_E107.2; no longer U402.12 (CC1)
- net CC2: now also R_E105.1; no longer DS1.5 (COMMON_CATHODE_DIGIT_2)
- net CC22: now also R_E108.2; no longer U402.9 (CC2)
- net CC3: now also R_E106.1; no longer DS1.7 (COMMON_CATHODE_DIGIT_3)
- net CC33: now also R_E109.2; no longer U402.8 (CC3)
- net CC44: now also R_E110.2; no longer U402.6 (CC4)
- net CCL123: now also R_E103.2; no longer DS1.14 (COMMON_CATHODE__L1L2L3)
- net a: now also R_E111.1
- net b: now also R_E112.1
- net c: now also R_E113.1
- new net: DS1.5 (COMMON_CATHODE_DIGIT_2), R_E105.2
- new net: DS1.1 (COMMON_CATHODE_DIGIT_1), R_E104.2
- new net: DS1.14 (COMMON_CATHODE__L1L2L3), R_E103.1
- new net: DS1.7 (COMMON_CATHODE_DIGIT_3), R_E106.2
- new net: R_E108.1, U402.9 (CC2)
- new net: R_E107.1, U402.12 (CC1)
- new net: R_E109.1, U402.8 (CC3)
- new net: D8.1 (K), R_E111.2, R_E112.2, R_E113.2
- new net: R_E110.1, U402.6 (CC4)

Commit message: reworked the schematic, changed differential pairs and RF traces, small PCB adjustments
Parts:
- DS1: value *LTC-4724JF -> LTC-4724JF; footprint Display_7Segment:LTC4724JF -> KiCad:LTC4724JF
Changed lines of the file:
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@@
+	(wire
+		(pts
+			(xy 165.1 187.96) (xy 161.29 187.96)
+		)
+		(stroke
+			(width 0)
+			(type default)
+		)
+	)
 	(wire
 		(pts
@@
 		(shape bidirectional)
 		(at 124.46 59.69 0)
+		(effects
+			(font
+				(size 1.27 1.27)
+			)
+			(justify left)
+		)
+	)
+	(hierarchical_label "5V"
+		(shape input)
+		(at 165.1 187.96 0)
 		(effects
 			(font
@@
 			)
 		)
-		(property "Value" "*LTC-4724JF"
+		(property "Value" "LTC-4724JF"
 			(at 100.33 130.81 0)
 			(show_name no)
@@
 			)
 		)
-		(property "Footprint" "Display_7Segment:LTC4724JF"
+		(property "Footprint" "KiCad:LTC4724JF"
 			(at 134.62 230.81 0)
 			(hide yes)
@@
 					(unit 1)
 				)
+			)
+		)
+	)
+	(symbol
+		(lib_id "power:+5V")
+		(at 161.29 187.96 90)
+		(unit 1)
+		(body_style 1)
+		(exclude_from_sim no)
+		(in_bom yes)
+		(on_board yes)
+		(in_pos_files yes)
+		(dnp no)
+		(fields_autoplaced yes)
+		(property "Reference" "#PWR0429"
+			(at 165.1 187.96 0)
+			(hide yes)
+			(show_name no)
+			(do_not_autoplace no)
+			(effects
+				(font
+					(size 1.27 1.27)
+				)
+			)
+		)
+		(property "Value" "+5V"
+			(at 157.48 187.9599 90)
+			(show_name no)
+			(do_not_autoplace no)
+			(effects
+				(font
+					(size 1.27 1.27)
+				)
+				(justify left)
+			)
+		)
+		(property "Footprint" ""
+			(at 161.29 187.96 0)
+			(hide yes)
+			(show_name no)
+			(do_not_autoplace no)
+			(effects
+				(font
+					(size 1.27 1.27)
+				)
+			)
+		)
+		(property "Datasheet" ""
+			(at 161.29 187.96 0)
+			(hide yes)
+			(show_name no)
+			(do_not_autoplace no)
+			(effects
+				(font
+					(size 1.27 1.27)
+				)
+			)
+		)
+		(property "Description" "Power symbol creates a global label with name \"+5V\""
+			(at 161.29 187.96 0)
+			(hide yes)
+			(show_name no)
+			(do_not_autoplace no)
+			(effects
+				(font
+					(size 1.27 1.27)
+				)
+			)
+		)
+		(pin "1"
+		)
+		(instances
+			(project "gps"
+				(path "/00526ddc-5304-4072-af1e-192a9e7e83da/944a09ba-484a-42c8-9e47-79436575a39f"
+					(reference "#PWR0429")
+					(unit 1)
+				)
