File: V2_WIP/ESP.kicad_sch (KiCad schematic)
At the start: 34 parts, among them J202 USB4145-03-0230-C, Q1 IRLML5203, Q2 S8050, Q3 S8050, SW2 PTS647SN70SMTR2N LFS, U1 ESP32-WROOM-32UE, U14 *CH340K, U201 RT9080-33GJ5

Commit message: up to date i dont remember what changed
Parts:
- added C203: 1uF, Capacitor_SMD:C_0603_1608Metric_Pad1.08x0.95mm_HandSolder, symbol Device:C
- added C204: 10uF, Capacitor_SMD:C_0603_1608Metric_Pad1.08x0.95mm_HandSolder, symbol Device:C
Connections:
- net +3V3: now also C203.1, C204.1
- net GND: now also C203.2, C204.2
Other:
- moved on the sheet: C2
