File: V2_WIP/GNSS.kicad_sch (KiCad schematic)
At the start: 17 parts, among them J301 USB_B_Micro, U301 USBLC6-2SC6, U401 NEO-M9N

Commit message: updated most datashets
Parts:
- C401: value 10uF -> *10uF
- C403: value 10n -> 10nF
- J301: value USB_B_Micro -> *USB_B_Micro
- U401: value NEO-M9N -> *NEO-M9N
Changed lines of the file:
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@@
 			)
 		)
-		(property "Datasheet" "~"
+		(property "Datasheet" "https://cz.mouser.com/ProductDetail/Murata-Electronics/LQG15HS27NG02D?qs=d0WKAl%252BL4KbSxh2r%2Fhe7ig%3D%3D"
 			(at 179.07 104.14 0)
 			(effects
@@
 			)
 		)
+		(property "Purchase-URL" ""
+			(at 179.07 104.14 0)
+			(effects
+				(font
+					(size 1.27 1.27)
+				)
+				(hide yes)
+			)
+		)
 		(pin "1"
 		)
@@
 			)
 		)
-		(property "Datasheet" "https://www.st.com/resource/en/datasheet/usblc6-2.pdf"
+		(property "Datasheet" "https://cz.mouser.com/ProductDetail/STMicroelectronics/USBLC6-2SC6?qs=po45yt2pPpu%2FhNIlwQdTlg%3D%3D"
 			(at 87.63 102.235 0)
 			(effects
@@
 			)
 		)
+		(property "Purchase-URL" ""
+			(at 86.36 93.98 0)
+			(effects
+				(font
+					(size 1.27 1.27)
+				)
+				(hide yes)
+			)
+		)
 		(pin "3"
 		)
@@
 			)
 		)
+		(property "Purchase-URL" ""
+			(at 121.92 120.65 0)
+			(effects
+				(font
+					(size 1.27 1.27)
+				)
+				(hide yes)
+			)
+		)
 		(pin "1"
 		)
@@
 			)
 		)
-		(property "Datasheet" "~"
+		(property "Datasheet" "https://cz.mouser.com/ProductDetail/TAIYO-YUDEN/MAJCT168BB7105MTEA01?qs=ZcfC38r4PotuS6MgLmtX7A%3D%3D"
 			(at 163.83 66.04 0)
 			(effects
@@
 			)
 		)
+		(property "Purchase-URL" ""
+			(at 163.83 66.04 0)
+			(effects
+				(font
+					(size 1.27 1.27)
+				)
+				(hide yes)
+			)
+		)
 		(pin "1"
 		)
@@
 			)
 		)
-		(property "Datasheet" "~"
+		(property "Datasheet" "https://cz.mouser.com/ProductDetail/Taoglas/PCBSMAFRAHT?qs=RuW%2Fu%252BNMQmubIFYcN8w5Dw%3D%3D&mgh=1&utm_id=20233080446&utm_source=google&utm_medium=cpc&utm_marketing_tactic=emeacorp&gad_source=1&gad_campaignid=20233099895&gbraid=0AAAAADn_wf1mWtjLE4a_0dNs1qHbugm4y&gclid=Cj0KCQjw18bEBhCBARIsAKuAFEZn-SykdQloeQqUWGMBdWb9HChtoLlFsgV0SERtX0LgUwmCsr2lQ1waAiK5EALw_wcB"
 			(at 209.55 88.9 0)
 			(effects
@@
 			)
 		)
+		(property "Purchase-URL" ""
+			(at 209.55 91.44 0)
+			(effects
+				(font
+					(size 1.27 1.27)
+				)
+				(hide yes)
+			)
+		)
 		(pin "1"
 		)
@@
 			)
 		)
-		(property "Datasheet" "~"
+		(property "Datasheet" "https://cz.mouser.com/ProductDetail/TAIYO-YUDEN/MAJCT168BB7105MTEA01?qs=ZcfC38r4PotuS6MgLmtX7A%3D%3D"
 			(at 124.46 77.47 0)
 			(effects
@@
 			)
 		)
+		(property "Purchase-URL" ""
+			(at 124.46 77.47 0)
+			(effects
+				(font
+					(size 1.27 1.27)
+				)
+				(hide yes)
+			)
+		)
 		(pin "1"
 		)
@@
 			)
 		)
-		(property "Datasheet" "~"
+		(property "Datasheet" "https://cz.mouser.com/ProductDetail/Wurth-Elektronik/636101112001?qs=iLbezkQI%252BshOHZpPZv%252BznA%3D%3D&mgh=1&utm_id=20233080446&utm_source=google&utm_medium=cpc&utm_marketing_tactic=emeacorp&gad_source=1&gad_campaignid=20233099895&gbraid=0AAAAADn_wf1mWtjLE4a_0dNs1qHbugm4y&gclid=Cj0KCQjw18bEBhCBARIsAKuAFEbAXKSMiM8PIGinrVoNUTtwBZcT9SeC7vJE1Ug8STwrMHge5dS1ieAaAhgVEALw_wcB"
 			(at 189.23 88.9 0)
 			(effects
@@
 			)
 		)
+		(property "Purchase-URL" ""
+			(at 189.23 91.44 0)
+			(effects
+				(font
+					(size 1.27 1.27)
+				)
+				(hide yes)
+			)
+		)
 		(pin "1"
 		)
@@
 			)
 		)
-		(property "Datasheet" "~"
+		(property "Datasheet" "https://cz.mouser.com/ProductDetail/Vishay/CRCW06030000Z0EI?qs=sGAEpiMZZMtlubZbdhIBIKbhzOdzan%2FG0ZM4rsijxcU%3D"
 			(at 139.7 73.66 0)
 			(effects
@@
 			)
 		)
+		(property "Purchase-URL" ""
+			(at 139.7 73.66 0)
+			(effects
+				(font
+					(size 1.27 1.27)
+				)
+				(hide yes)
+			)
+		)
 		(pin "2"
 		)
@@
 			)
 		)
+		(property "Purchase-URL" ""
+			(at 119.38 97.79 0)
+			(effects
+				(font
+					(size 1.27 1.27)
+				)
+				(hide yes)
+			)
+		)
 		(pin "1"
 		)
@@
 			)
 		)
-		(property "Value" "NEO-M9N"
+		(property "Value" "*NEO-M9N"
 			(at 141.8941 133.35 0)
 			(effects
@@
 			)
 		)
+		(property "Purchase-URL" ""
+			(at 139.7 107.95 0)
+			(effects
+				(font
+					(size 1.27 1.27)
+				)
+				(hide yes)
+			)
+		)
 		(pin "1"
 		)
@@
 			)
 		)
-		(property "Value" "10uF"
+		(property "Value" "*10uF"
 			(at 154.94 66.4209 0)
 			(effects
@@
 			)
 		)
-		(property "Datasheet" "~"
+		(property "Datasheet" ""
 			(at 151.13 66.04 0)
 			(effects
@@
 			)
 		)
+		(property "Purchase-URL" ""
+			(at 151.13 66.04 0)
+			(effects
+				(font
+					(size 1.27 1.27)
+				)
+				(hide yes)
+			)
+		)
 		(pin "1"
 		)
@@
 			)
 		)
+		(property "Purchase-URL" ""
+			(at 76.2 82.55 0)
+			(effects
+				(font
+					(size 1.27 1.27)
+				)
+				(hide yes)
+			)
+		)
 		(pin "1"
 		)
@@
 			)
 		)
-		(property "Value" "USB_B_Micro"
+		(property "Value" "*USB_B_Micro"
 			(at 57.15 83.82 0)
 			(effects
@@
 			)
 		)
-		(property "Datasheet" "https://cz.mouser.com/datasheet/2/837/USB3145-2888215.pdf"
+		(property "Datasheet" ""
 			(at 60.96 95.25 0)
 			(effects
@@
 			)
 		)
+		(property "Purchase-URL" ""
+			(at 57.15 93.98 0)
+			(effects
+				(font
+					(size 1.27 1.27)
+				)
+				(hide yes)
+			)
+		)
 		(pin "1"
 		)
@@
 			)
 		)
-		(property "Value" "10n"
+		(property "Value" "10nF"
 			(at 172.72 95.25 90)
 			(effects
@@
 			)
 		)
-		(property "Datasheet" "~"
+		(property "Datasheet" "https://cz.mouser.com/ProductDetail/KYOCERA-AVX/KAM21BR71H103KT?qs=OcgtsXO%252B3gswRpZaaXH9DQ%3D%3D"
 			(at 172.72 100.33 0)
 			(effects
@@
 			)
 		)
+		(property "Purchase-URL" ""
+			(at 172.72 100.33 0)
+			(effects
+				(font
+					(size 1.27 1.27)
+				)
+				(hide yes)
+			)
+		)
 		(pin "1"
 		)
@@
 			)
 		)
+		(property "Purchase-URL" ""
+			(at 119.38 106.68 0)
+			(effects
+				(font
+					(size 1.27 1.27)
+				)
+				(hide yes)
+			)
+		)
 		(pin "1"
 		)
@@
 			)
 		)
+		(property "Purchase-URL" ""
+			(at 110.49 78.74 0)
+			(effects
+				(font
+					(size 1.27 1.27)
+				)
+				(hide yes)
+			)
+		)
 		(pin "1"
 		)
@@
 			)
 		)
-		(property "Datasheet" "~"
+		(property "Datasheet" "https://cz.mouser.com/ProductDetail/Vishay-Beyschlag/MCT06030C1009FP500?qs=sGAEpiMZZMtlubZbdhIBIOZdEduus70kc745foTe5h0%3D"
 			(at 179.07 92.71 0)
 			(effects
@@
 			(at 179.07 92.71 0)
 			(effects
+				(font
+					(size 1.27 1.27)
+				)
+				(hide yes)
+			)
+		)
+		(property "Purchase-URL" ""
+			(at 179.07 92.71 0)
+			(effects

Commit message: up to date i dont remember what changed
Changed lines of the file:
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@@
 (kicad_sch
-	(version 20231120)
+	(version 20250114)
 	(generator "eeschema")
-	(generator_version "8.0")
+	(generator_version "9.0")
 	(paper "A4")
 	(junction
@@
 		(shape input)
 		(at 111.76 102.87 180)
-		(fields_autoplaced yes)
 		(effects
 			(font
@@
 		(shape output)
 		(at 76.2 77.47 90)
-		(fields_autoplaced yes)
 		(effects
 			(font
@@
 		(shape output)
 		(at 157.48 115.57 0)
-		(fields_autoplaced yes)
 		(effects
 			(font
@@
 		(shape output)
 		(at 111.76 100.33 180)
-		(fields_autoplaced yes)
 		(effects
 			(font
